File: capbot.sch (EAGLE design)
At the start: 46 parts, among them J1 USBPCB, J2 USBPCB, J3 USBPCB

Commit message: r1
Parts:
- LED1, LED2, LED3, LED4, LED5, LED6: device led:LED3MM -> cwpackage:LED3MM-MOREFLAT
Changed lines of the file:
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@@
 <grid distance="0.1" unitdist="inch" unit="inch" style="lines" multiple="1" display="no" altdistance="0.01" altunitdist="inch" altunit="inch"/>
 <layers>
-<layer number="1" name="Top" color="4" fill="1" visible="no" active="no"/>
-<layer number="16" name="Bottom" color="1" fill="1" visible="no" active="no"/>
-<layer number="17" name="Pads" color="2" fill="1" visible="no" active="no"/>
-<layer number="18" name="Vias" color="2" fill="1" visible="no" active="no"/>
-<layer number="19" name="Unrouted" color="6" fill="1" visible="no" active="no"/>
-<layer number="20" name="Dimension" color="15" fill="1" visible="no" active="no"/>
-<layer number="21" name="tPlace" color="7" fill="1" visible="no" active="no"/>
-<layer number="22" name="bPlace" color="7" fill="1" visible="no" active="no"/>
-<layer number="23" name="tOrigins" color="15" fill="1" visible="no" active="no"/>
-<layer number="24" name="bOrigins" color="15" fill="1" visible="no" active="no"/>
-<layer number="25" name="tNames" color="7" fill="1" visible="no" active="no"/>
-<layer number="26" name="bNames" color="7" fill="1" visible="no" active="no"/>
-<layer number="27" name="tValues" color="7" fill="1" visible="no" active="no"/>
-<layer number="28" name="bValues" color="7" fill="1" visible="no" active="no"/>
+<layer number="1" name="Top" color="4" fill="1" visible="yes" active="no"/>
+<layer number="16" name="Bottom" color="1" fill="1" visible="yes" active="no"/>
+<layer number="17" name="Pads" color="2" fill="1" visible="yes" active="no"/>
+<layer number="18" name="Vias" color="2" fill="1" visible="yes" active="no"/>
+<layer number="19" name="Unrouted" color="6" fill="1" visible="yes" active="no"/>
+<layer number="20" name="Dimension" color="15" fill="1" visible="yes" active="no"/>
+<layer number="21" name="tPlace" color="7" fill="1" visible="yes" active="no"/>
+<layer number="22" name="bPlace" color="7" fill="1" visible="yes" active="no"/>
+<layer number="23" name="tOrigins" color="15" fill="1" visible="yes" active="no"/>
+<layer number="24" name="bOrigins" color="15" fill="1" visible="yes" active="no"/>
+<layer number="25" name="tNames" color="7" fill="1" visible="yes" active="no"/>
+<layer number="26" name="bNames" color="7" fill="1" visible="yes" active="no"/>
+<layer number="27" name="tValues" color="7" fill="1" visible="yes" active="no"/>
+<layer number="28" name="bValues" color="7" fill="1" visible="yes" active="no"/>
 <layer number="29" name="tStop" color="7" fill="3" visible="no" active="no"/>
 <layer number="30" name="bStop" color="7" fill="6" visible="no" active="no"/>
@@
 <layer number="35" name="tGlue" color="7" fill="4" visible="no" active="no"/>
 <layer number="36" name="bGlue" color="7" fill="5" visible="no" active="no"/>
-<layer number="37" name="tTest" color="7" fill="1" visible="no" active="no"/>
-<layer number="38" name="bTest" color="7" fill="1" visible="no" active="no"/>
+<layer number="37" name="tTest" color="7" fill="1" visible="yes" active="no"/>
+<layer number="38" name="bTest" color="7" fill="1" visible="yes" active="no"/>
 <layer number="39" name="tKeepout" color="4" fill="11" visible="no" active="no"/>
 <layer number="40" name="bKeepout" color="1" fill="11" visible="no" active="no"/>
@@
 <layer number="44" name="Drills" color="7" fill="1" visible="no" active="no"/>
 <layer number="45" name="Holes" color="7" fill="1" visible="no" active="no"/>
-<layer number="46" name="Milling" color="3" fill="1" visible="no" active="no"/>
-<layer number="47" name="Measures" color="7" fill="1" visible="no" active="no"/>
-<layer number="48" name="Document" color="7" fill="1" visible="no" active="no"/>
-<layer number="49" name="Reference" color="7" fill="1" visible="no" active="no"/>
-<layer number="50" name="dxf" color="7" fill="1" visible="no" active="no"/>
-<layer number="51" name="tDocu" color="7" fill="1" visible="no" active="no"/>
-<layer number="52" name="bDocu" color="7" fill="1" visible="no" active="no"/>
-<layer number="53" name="tGND_GNDA" color="7" fill="9" visible="no" active="no"/>
-<layer number="54" name="bGND_GNDA" color="1" fill="9" visible="no" active="no"/>
-<layer number="56" name="wert" color="7" fill="1" visible="no" active="no"/>
-<layer number="57" name="tCAD" color="7" fill="1" visible="no" active="no"/>
-<layer number="59" name="tCarbon" color="7" fill="1" visible="no" active="no"/>
-<layer number="60" name="bCarbon" color="7" fill="1" visible="no" active="no"/>
+<layer number="46" name="Milling" color="3" fill="1" visible="yes" active="no"/>
+<layer number="47" name="Measures" color="7" fill="1" visible="yes" active="no"/>
+<layer number="48" name="Document" color="7" fill="1" visible="yes" active="no"/>
+<layer number="49" name="Reference" color="7" fill="1" visible="yes" active="no"/>
+<layer number="50" name="dxf" color="7" fill="1" visible="yes" active="no"/>
+<layer number="51" name="tDocu" color="7" fill="1" visible="yes" active="no"/>
+<layer number="52" name="bDocu" color="7" fill="1" visible="yes" active="no"/>
+<layer number="53" name="tGND_GNDA" color="7" fill="9" visible="yes" active="no"/>
+<layer number="54" name="bGND_GNDA" color="1" fill="9" visible="yes" active="no"/>
+<layer number="56" name="wert" color="7" fill="1" visible="yes" active="no"/>
+<layer number="57" name="tCAD" color="7" fill="1" visible="yes" active="no"/>
+<layer number="59" name="tCarbon" color="7" fill="1" visible="yes" active="no"/>
+<layer number="60" name="bCarbon" color="7" fill="1" visible="yes" active="no"/>
 <layer number="90" name="Modules" color="5" fill="1" visible="yes" active="yes"/>
 <layer number="91" name="Nets" color="2" fill="1" visible="yes" active="yes"/>
@@
 <part name="C2" library="resistor" deviceset="C-EU" device="C1206"/>
 <part name="IC1" library="adafruit" deviceset="MCP1700" device="INLINE"/>
-<part name="LED1" library="led" deviceset="LED" device="3MM"/>
-<part name="LED2" library="led" deviceset="LED" device="3MM"/>
+<part name="LED1" library="cwpackage" deviceset="LED" device="3MM-MOREFLAT"/>
+<part name="LED2" library="cwpackage" deviceset="LED" device="3MM-MOREFLAT"/>
 <part name="JP2" library="pinhead" deviceset="PINHD-1X4" device=""/>
 <part name="J1" library="SparkFun-Connectors" deviceset="USB" device="PCB"/>
@@
 <part name="C4" library="resistor" deviceset="C-EU" device="C1206"/>
 <part name="IC2" library="adafruit" deviceset="MCP1700" device="INLINE"/>
-<part name="LED3" library="led" deviceset="LED" device="3MM"/>
-<part name="LED4" library="led" deviceset="LED" device="3MM"/>
+<part name="LED3" library="cwpackage" deviceset="LED" device="3MM-MOREFLAT"/>
+<part name="LED4" library="cwpackage" deviceset="LED" device="3MM-MOREFLAT"/>
 <part name="JP4" library="pinhead" deviceset="PINHD-1X4" device=""/>
 <part name="J2" library="SparkFun-Connectors" deviceset="USB" device="PCB"/>
@@
 <part name="C7" library="resistor" deviceset="C-EU" device="C1206"/>
 <part name="IC3" library="adafruit" deviceset="MCP1700" device="INLINE"/>
-<part name="LED5" library="led" deviceset="LED" device="3MM"/>
-<part name="LED6" library="led" deviceset="LED" device="3MM"/>
+<part name="LED5" library="cwpackage" deviceset="LED" device="3MM-MOREFLAT"/>
+<part name="LED6" library="cwpackage" deviceset="LED" device="3MM-MOREFLAT"/>
 <part name="JP6" library="pinhead" deviceset="PINHD-1X4" device=""/>
 <part name="J3" library="SparkFun-Connectors" deviceset="USB" device="PCB"/>

Commit message: Move the pin header 0.8 mm closer to the edge so that the horizontal part of the wires can sit flush to the surface with less bending and filing.
This required changing the pads from "long" to "offset" to prevent them from getting too close to the edge. Unfortunately it seems a pad can only be offset all the way, the drill position is not continuously adjustable - I'd have preferred something in between.
Parts:
- JP2, JP4, JP6: device pinhead:PINHD-1X4 -> cwpinhead:PINHD-1X4
Changed lines of the file:
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@@
 <part name="LED1" library="cwpackage" deviceset="LED" device="3MM-MOREFLAT"/>
 <part name="LED2" library="cwpackage" deviceset="LED" device="3MM-MOREFLAT"/>
-<part name="JP2" library="pinhead" deviceset="PINHD-1X4" device=""/>
+<part name="JP2" library="cwpinhead" deviceset="PINHD-1X4" device=""/>
 <part name="J1" library="SparkFun-Connectors" deviceset="USB" device="PCB"/>
 <part name="S2" library="switch" deviceset="TL36PO" device="" value=""/>
@@
 <part name="LED3" library="cwpackage" deviceset="LED" device="3MM-MOREFLAT"/>
 <part name="LED4" library="cwpackage" deviceset="LED" device="3MM-MOREFLAT"/>
-<part name="JP4" library="pinhead" deviceset="PINHD-1X4" device=""/>
+<part name="JP4" library="cwpinhead" deviceset="PINHD-1X4" device=""/>
 <part name="J2" library="SparkFun-Connectors" deviceset="USB" device="PCB"/>
 <part name="C5" library="resistor" deviceset="CPOL-EU" device="E5-10.5"/>
@@
 <part name="LED5" library="cwpackage" deviceset="LED" device="3MM-MOREFLAT"/>
 <part name="LED6" library="cwpackage" deviceset="LED" device="3MM-MOREFLAT"/>
-<part name="JP6" library="pinhead" deviceset="PINHD-1X4" device=""/>
+<part name="JP6" library="cwpinhead" deviceset="PINHD-1X4" device=""/>
 <part name="J3" library="SparkFun-Connectors" deviceset="USB" device="PCB"/>
 </parts>
