File: capbot.sch (EAGLE design)
At the start: 46 parts, among them J1 USBPCB, J2 USBPCB, J3 USBPCB

Commit message: Add power LED function.
With one added Zener diode, the top LED indicates that the device is powered, while both LEDs together still indicate that charging is completed.
Parts:
- added D1, D2, D3: BZX55/6, cwpackage:BZX55/6
- R2, R4, R6: device resistor:R-EU_0207/5V -> resistor:R-EU_0207/7
Connections:
- net N$14: now also D3.A
- net N$19: now also D3.C
- net N$24: now also D2.A
- net N$29: now also D2.C
- net N$4: now also D1.A
- net N$9: now also D1.C
Changed lines of the file:
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@@
 <part name="PAD4" library="wirepad" deviceset="WIREPAD" device="2,15/1,0"/>
 <part name="R1" library="resistor" deviceset="R-EU_" device="0207/7"/>
-<part name="R2" library="resistor" deviceset="R-EU_" device="0207/5V"/>
+<part name="R2" library="resistor" deviceset="R-EU_" device="0207/7"/>
 <part name="C2" library="resistor" deviceset="C-EU" device="C1206"/>
 <part name="IC1" library="adafruit" deviceset="MCP1700" device="INLINE"/>
@@
 <part name="PAD8" library="wirepad" deviceset="WIREPAD" device="2,15/1,0"/>
 <part name="R3" library="resistor" deviceset="R-EU_" device="0207/7"/>
-<part name="R4" library="resistor" deviceset="R-EU_" device="0207/5V"/>
+<part name="R4" library="resistor" deviceset="R-EU_" device="0207/7"/>
 <part name="C4" library="resistor" deviceset="C-EU" device="C1206"/>
 <part name="IC2" library="adafruit" deviceset="MCP1700" device="INLINE"/>
@@
 <part name="PAD12" library="wirepad" deviceset="WIREPAD" device="2,15/1,0"/>
 <part name="R5" library="resistor" deviceset="R-EU_" device="0207/7"/>
-<part name="R6" library="resistor" deviceset="R-EU_" device="0207/5V"/>
+<part name="R6" library="resistor" deviceset="R-EU_" device="0207/7"/>
 <part name="C7" library="resistor" deviceset="C-EU" device="C1206"/>
 <part name="IC3" library="adafruit" deviceset="MCP1700" device="INLINE"/>
@@
 <part name="JP6" library="cwpinhead" deviceset="PINHD-1X4" device=""/>
 <part name="J3" library="SparkFun-Connectors" deviceset="USB" device="PCB"/>
+<part name="D1" library="cwpackage" deviceset="BZX55" device="/6"/>
+<part name="D2" library="cwpackage" deviceset="BZX55" device="/6"/>
+<part name="D3" library="cwpackage" deviceset="BZX55" device="/6"/>
 </parts>
 <sheets>
@@
 <instance part="JP6" gate="A" x="71.12" y="60.96"/>
 <instance part="J3" gate="G$1" x="10.16" y="68.58" rot="R180"/>
+<instance part="D1" gate="1" x="43.18" y="22.86"/>
+<instance part="D2" gate="1" x="43.18" y="71.12"/>
+<instance part="D3" gate="1" x="43.18" y="121.92"/>
 </instances>
 <busses>
@@
 <pinref part="LED2" gate="G$1" pin="A"/>
 <wire x1="53.34" y1="17.78" x2="53.34" y2="20.32" width="0.1524" layer="91"/>
+<pinref part="D1" gate="1" pin="C"/>
+<wire x1="45.72" y1="22.86" x2="48.26" y2="22.86" width="0.1524" layer="91"/>
+<wire x1="48.26" y1="22.86" x2="48.26" y2="20.32" width="0.1524" layer="91"/>
+<wire x1="48.26" y1="20.32" x2="53.34" y2="20.32" width="0.1524" layer="91"/>
+<junction x="53.34" y="20.32"/>
 </segment>
 </net>
@@
 <pinref part="R1" gate="G$1" pin="1"/>
 <wire x1="12.7" y1="20.32" x2="17.78" y2="20.32" width="0.1524" layer="91"/>
+<pinref part="D1" gate="1" pin="A"/>
+<wire x1="40.64" y1="22.86" x2="17.78" y2="22.86" width="0.1524" layer="91"/>
+<wire x1="17.78" y1="22.86" x2="17.78" y2="20.32" width="0.1524" layer="91"/>
+<junction x="17.78" y="20.32"/>
 </segment>
 </net>
@@
 <pinref part="LED4" gate="G$1" pin="A"/>
 <wire x1="53.34" y1="116.84" x2="53.34" y2="119.38" width="0.1524" layer="91"/>
+<pinref part="D3" gate="1" pin="C"/>
+<wire x1="45.72" y1="121.92" x2="48.26" y2="121.92" width="0.1524" layer="91"/>
+<wire x1="48.26" y1="121.92" x2="48.26" y2="119.38" width="0.1524" layer="91"/>
+<wire x1="48.26" y1="119.38" x2="53.34" y2="119.38" width="0.1524" layer="91"/>
+<junction x="53.34" y="119.38"/>
 </segment>
 </net>
@@
 <pinref part="R3" gate="G$1" pin="1"/>
 <wire x1="12.7" y1="119.38" x2="17.78" y2="119.38" width="0.1524" layer="91"/>
+<pinref part="D3" gate="1" pin="A"/>
+<wire x1="40.64" y1="121.92" x2="17.78" y2="121.92" width="0.1524" layer="91"/>
+<wire x1="17.78" y1="121.92" x2="17.78" y2="119.38" width="0.1524" layer="91"/>
+<junction x="17.78" y="119.38"/>
 </segment>
 </net>
@@
 <pinref part="LED6" gate="G$1" pin="A"/>
 <wire x1="53.34" y1="66.04" x2="53.34" y2="68.58" width="0.1524" layer="91"/>
+<pinref part="D2" gate="1" pin="C"/>
+<wire x1="45.72" y1="71.12" x2="48.26" y2="71.12" width="0.1524" layer="91"/>
+<wire x1="48.26" y1="71.12" x2="48.26" y2="68.58" width="0.1524" layer="91"/>
+<wire x1="48.26" y1="68.58" x2="53.34" y2="68.58" width="0.1524" layer="91"/>
+<junction x="53.34" y="68.58"/>
 </segment>
 </net>
@@
 <pinref part="R5" gate="G$1" pin="1"/>
 <wire x1="12.7" y1="68.58" x2="17.78" y2="68.58" width="0.1524" layer="91"/>
-</segment>
-</net>
+<pinref part="D2" gate="1" pin="A"/>
+<wire x1="40.64" y1="71.12" x2="17.78" y2="71.12" width="0.1524" layer="91"/>
+<wire x1="17.78" y1="71.12" x2="17.78" y2="68.58" width="0.1524" layer="91"/>
+<junction x="17.78" y="68.58"/>
+</segment>
+</net>
